File: analog_shield.kicad_pcb (KiCad board)
At the start: 4 copper layers, 68.6 x 53.3 mm, 49 parts, among them J1 640456-3, J2 S3B-EH(LF)(SN), J3 Conn_01x08, J4 Conn_01x06, J6 Conn_01x10, J7 Conn_01x08, J8 PPTC062LFBN-RC, U1 LMT84LPM, U2 TLV2472AIP

Commit message: Updated Title block with correct information, all documentation updated too.
Connections:
- net +3V3 renamed +3.3V

Commit message: Documentation and GitHub pages update.
Other:
- board text added: "LAYER 1"
- board text added: "LAYER 2"
- board text added: "LAYER 3"
- board text added: "LAYER 4"
- board text removed: "0.2500 mm / 0.0000 mm"
- board text removed: "0.3000 mm"
- board text removed: "1.6000 mm"
- board text removed: "4"
- board text removed: "68.5800 mm x 53.3400 mm"
- board text removed: "BOARD CHARACTERISTICS"
- board text removed: "Board Thickness:"
- board text removed: "Board overall dimensions:"
- board text removed: "Castellated pads:"
- board text removed: "Copper Finish:"
- board text removed: "Copper Layer Count:"
- board text removed: "Edge card connectors:"
- board text removed: "HAL lead-free"
- board text removed: "Impedance Control:"
- board text removed: "Min hole diameter:"
- board text removed: "Min track/spacing:"
- board text removed: "No"
- board text removed: "Plated Board Edge:"
