File: analog_shield.kicad_sch (KiCad schematic)
At the start: 48 parts, among them J1 640456-3, J2 S3B-EH(LF)(SN), J3 Conn_01x08, J4 Conn_01x06, J6 Conn_01x10, J7 Conn_01x08, J8 PPTC062LFBN-RC, U1 LMT84LPM, U2 TLV2472AIP

Commit message: Updated Title block with correct information, all documentation updated too.
Other:
- company: (none) -> University of Toronto, Dept. of Physics E.S.S.
- title: (none) -> Analog Shield
Changed lines of the file:
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@@
 	(generator_version "10.0")
 	(paper "B")
+	(title_block
+		(title "Analog Shield")
+		(date "2023-05-04")
+		(rev "C")
+		(company "University of Toronto, Dept. of Physics E.S.S.")
+	)
 	(rectangle
 		(start 229.87 124.46)

Commit message: Documentation and GitHub pages update.
Parts:
- H1, H2, H3, H4: now left out of the parts list
Changed lines of the file:
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@@
 		(unit 1)
 		(body_style 1)
-		(exclude_from_sim no)
-		(in_bom yes)
+		(exclude_from_sim yes)
+		(in_bom no)
 		(on_board yes)
-		(in_pos_files yes)
+		(in_pos_files no)
 		(dnp no)
 		(fields_autoplaced yes)
@@
 		(unit 1)
 		(body_style 1)
-		(exclude_from_sim no)
-		(in_bom yes)
+		(exclude_from_sim yes)
+		(in_bom no)
 		(on_board yes)
-		(in_pos_files yes)
+		(in_pos_files no)
 		(dnp no)
 		(fields_autoplaced yes)
@@
 		(unit 1)
 		(body_style 1)
-		(exclude_from_sim no)
-		(in_bom yes)
+		(exclude_from_sim yes)
+		(in_bom no)
 		(on_board yes)
-		(in_pos_files yes)
+		(in_pos_files no)
 		(dnp no)
 		(fields_autoplaced yes)
@@
 		(unit 1)
 		(body_style 1)
-		(exclude_from_sim no)
-		(in_bom yes)
+		(exclude_from_sim yes)
+		(in_bom no)
 		(on_board yes)
-		(in_pos_files yes)
+		(in_pos_files no)
 		(dnp no)
 		(fields_autoplaced yes)
